File: PCB/LED panel/LED panel.kicad_sch (KiCad schematic)
At the start: 20 parts

Commit message: LED panel PCB!
Parts:
- removed D11, D12, D13, D14, D15, D16, D17, D18, D19, D20: WS2812B, LED_SMD:LED_WS2812B_PLCC4_5.0x5.0mm_P3.2mm, symbol LED:WS2812B
