File: PCB/core/core.kicad_sch (KiCad schematic)
At the start: 9 parts, among them U1 MCU_Seeed_XIAO_ESP32-C3, U2 STP55NF06L

Commit message: im tired
Connections:
- net M_GND is gone; now on net A3144E GND: U2.3
- net GND renamed A3144E GND
