File: PCB/core/core.kicad_pcb (KiCad board)
At the start: 2 copper layers, 100 x 100 mm, 39 parts, among them U1 MCU_Seeed_XIAO_ESP32-C3, U2 STP55NF06L

Commit message: 07012025 - pcb updates and some cad work!
Parts:
- moved D1 6.32 mm to (168.4, 112.0)
- moved D2 3.66 mm to (174.0, 97.7), turned to -90 degrees
- moved R1 1.68 mm to (174.0, 92.3)
Routing:
- net Net-(D2-A): track 31.6 -> 38.9 mm
- net Net-(D1-K): track 18.0 -> 24.1 mm
- net A3114E POW: track 308.9 -> 311.8 mm
- net MOTOR-: track 33.9 -> 35.6 mm
- net A3144E GND: track 294.4 -> 295.2 mm
- net Net-(R1-Pad2): track 7.48 -> 6.79 mm
- net Net-(D2-K): track 4.90 -> 4.37 mm
Other:
- outline, holes or cut-outs redrawn
- board text added: "GND"
- board text added: "GPIO"
- board text added: "POW"
