File: PCB/core/_autosave-core.kicad_pcb (KiCad board)
At the start: 2 copper layers, 100 x 100 mm, 43 parts, among them U1 MCU_Seeed_XIAO_ESP32-C3, U2 STP55NF06L

Commit message: licenses!
Other:
- board text added: "A HackClub Highway Project!"
- board text added: "CORE PCB V.1"
- board text added: "RAVEN"
